File: Isolated_Gate_Driver.kicad_pcb (KiCad board)
At the start: 2 copper layers, 37.5 x 20 mm, 20 parts, among them J1 Conn_01x03_Pin, J2 tp, J3 Conn_01x02_Pin, U3 SN6505BDBV

Commit message: :uwu:
Changed lines of the file:
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@@
 		)
+	)
+	(gr_arc
+		(start 128.995356 71.486477)
+		(mid 128.383687 72.529184)
+		(end 127.459431 71.75)
+		(stroke
+			(width 0.2)
+			(type default)
+		)
+		(layer "F.Cu")
+	)
+	(gr_arc
+		(start 127.459431 71.75)
+		(mid 126.535175 72.529184)
+		(end 125.923506 71.486477)
+		(stroke
+			(width 0.2)
+			(type default)
+		)
+		(layer "F.Cu")
+	)
+	(gr_circle
+		(center 130 70)
+		(end 130.75 70.5)
+		(stroke
+			(width 0.2)
+			(type default)
+		)
+		(fill no)
+		(layer "F.Cu")
+	)
+	(gr_circle
+		(center 125 70)
+		(end 125.75 70.5)
+		(stroke
+			(width 0.2)
+			(type default)
+		)
+		(fill no)
+		(layer "F.Cu")
 	)
 	(gr_rect
